File: kaimat/kaimat.sch (KiCad schematic (older format))
At the start: 25 parts, among them J1 AudioJack2_Ground, J2 AudioJack2_Ground, J3 AudioJack2_Ground, J4 AudioJack2_Ground, SW1 Rotary_Encoder_Switch, SW2 Rotary_Encoder_Switch, SW3 SW_DIP_x02, SW4 SW_DIP_x02, U1 Waveshare_128x128_OLED_SSD1327, U2 Adafruit_NeoTrellis

Commit message: changed teensy 3.2 to 3.6
Parts:
- removed MCU1: Teensy3.2, symbol KaimatKicadLib:Teensy3.2
Changed lines of the file:
@@
 Text GLabel 10700 1450 2    50   Input ~ 0
 cvIn4
-Text GLabel 5450 6350 0    50   Input ~ 0
-GND
-Text GLabel 5450 6450 0    50   Input ~ 0
-enc1button
-Text GLabel 5450 6550 0    50   Input ~ 0
-enc1pinA
-Text GLabel 5450 6650 0    50   Input ~ 0
-enc1pinB
-Text GLabel 5450 7650 0    50   Input ~ 0
-b2
-Text GLabel 5450 7250 0    50   Input ~ 0
-OLEDreset
-Text GLabel 5450 7350 0    50   Input ~ 0
-OLEDdc
-Text GLabel 5450 7450 0    50   Input ~ 0
-OLEDcs
-Text GLabel 5450 7550 0    50   Input ~ 0
-OLEDdata
-Text GLabel 5450 6750 0    50   Input ~ 0
-DACdataout
-Text GLabel 5450 6850 0    50   Input ~ 0
-DACspiclk
-Text GLabel 5450 6950 0    50   Input ~ 0
-DACslaveSelect
-Text GLabel 5450 7050 0    50   Input ~ 0
-DACldac
-Text GLabel 5450 7150 0    50   Input ~ 0
-DACclr
-Text GLabel 6450 6650 2    50   Input ~ 0
-cvIn1
-Text GLabel 6450 6750 2    50   Input ~ 0
-cvIn2
-Text GLabel 6450 6850 2    50   Input ~ 0
-cvIn3
-Text GLabel 6450 7550 2    50   Input ~ 0
-enc2button
-Text GLabel 6450 7450 2    50   Input ~ 0
-enc2pinA
-Text GLabel 6450 7350 2    50   Input ~ 0
-enc2pinB
-Text GLabel 6450 7650 2    50   Input ~ 0
-OLEDclock
-Text GLabel 6450 7250 2    50   Input ~ 0
-b1
-Text GLabel 6450 7150 2    50   Input ~ 0
-trellisSDA
-Text GLabel 6450 7050 2    50   Input ~ 0
-trellisSCL
-Text GLabel 6450 6950 2    50   Input ~ 0
-cvIn4
-$Comp
-L KaimatKicadLib:Teensy3.2 MCU1
-U 1 1 5C680FB5
-P 5950 6200
-F 0 "MCU1" H 5950 6315 50  0000 C CNN
-F 1 "Teensy3.2" H 5950 6224 50  0000 C CNN
-F 2 "" H 5950 6350 50  0001 C CNN
-F 3 "" H 5950 6350 50  0001 C CNN
-	1    5950 6200
-	1    0    0    -1
-$EndComp
 $Comp
 L KaimatKicadLib:Teensy3.6 MCU2

Commit message: improved schem
Parts:
- removed D1, D2, D3, D4: DIODE, symbol pspice:DIODE
- added D? (x5): D_ALT, symbol Device:D_ALT
- added U?: Pin_Header_2x5, symbol eurocad:Pin_Header_2x5
Connections:
- net 3.3V is gone; now on net +3V3: U1.1 (VCC(Vin)), U2.4 (VIN)
- net 3.3v is gone; now on net +3V3: DAC1.3 (AVdd(Vin))
- net GND: now also J1.G, J2.G, J3.G, J4.G, MCU2.43 (AGND), R2.1, R4.1, R6.1, R8.1, U?.4 (GND), U?.6 (GND), U?.8 (GND)
- net cvIn1: now also D?.1 (K)
- net cvIn2: now also D?.1 (K)
- net cvIn3: now also D?.1 (K)
- net cvIn4: now also D?.1 (K)
- net at R1.1, R2.2: now also D?.2 (A)
- net at R3.1, R4.2: now also D?.2 (A)
- net at R5.1, R6.2: now also D?.2 (A)
- net at R7.1, R8.2: now also D?.2 (A)
- net +5V: now reaches MCU2.42 (VIN)
- net +3V3: now reaches MCU2.44 (3.3V)
- new net: D?.2 (A), U?.2 (+12V)
- new net VCC: D?.1 (K)
- no-connect marks 6 -> 16
Other:
- note added: "550"
- moved on the sheet: DAC1, J1, J2, J3, J4, MCU2, R1, R2, R3, R4, R5, R6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

Commit message: improved cod
Parts:
- added U?: LM1117-5.0, symbol Regulator_Linear:LM1117-5.0
Connections:
- net +3V3: no longer DAC1.3 (AVdd(Vin))
- net +5V: now also DAC1.3 (AVdd(Vin)), U?.2 (VO)
- net GND: now also SW3.2, SW4.2, U?.1 (GND)
- net b1: now also SW3.3
- net b2: now also SW4.3
- net TRout4: now reaches DAC1.10 (VoutH)
- net TRout2: now reaches DAC1.11 (VoutF)
- net CVout4: now reaches DAC1.12 (VoutD)
- net CVout2: now reaches DAC1.13 (VoutB)
- net CVout1: now reaches DAC1.4 (VoutA)
- net CVout3: now reaches DAC1.5 (VoutC)
- net TRout1: now reaches DAC1.6 (VoutE)
- net TRout3: now reaches DAC1.7 (VoutG)
- net VCC: no longer names the net of D?.1 (K)
- net VCC: now also U?.3 (VI)
- no-connect marks 16 -> 37
Other:
- moved on the sheet: D?, DAC1, J1, J2, J3, J4, R1, R2, R3, R4, R5, R6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
