File: Schematic/Eagle/KaiMat/kaimat.sch (EAGLE design)
At the start: 35 parts, among them IC1 MCP6004-E_P

Commit message: improved schematic
Parts:
- removed JP1: (no value), microbuilder:HEADER-1X5EDGESMT
- added U$4: NEOTRELLISKAIMAT2, Adafruit Trellis:NEOTRELLISKAIMAT2
- renumbered IC1 to OPAMP1
Connections:
- net +3V3: now also U$4.VIN
- net GND: now also U$4.GND
- net TRLSCL: now also U$4.SCL
- net TRLSDA: now also U$4.SDA
Changed lines of the file:
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@@
 <part name="S1" library="switch-omron" library_urn="urn:adsk.eagle:library:377" deviceset="10-XX" device="" package3d_urn="urn:adsk.eagle:package:27496/1"/>
 <part name="S2" library="switch-omron" library_urn="urn:adsk.eagle:library:377" deviceset="10-XX" device="" package3d_urn="urn:adsk.eagle:package:27496/1"/>
-<part name="JP1" library="microbuilder" deviceset="HEADER-1X5" device="EDGESMT"/>
 <part name="ENC2" library="switch-alps" library_urn="urn:adsk.eagle:library:373" deviceset="EC12E_SW" device="" package3d_urn="urn:adsk.eagle:package:27083/1"/>
 <part name="GND5" library="supply1" library_urn="urn:adsk.eagle:library:371" deviceset="GND" device=""/>
@@
 <part name="R1" library="MusicThingModular" deviceset="RESISTOR" device="7MM" value="100k"/>
 <part name="+3V2" library="supply1" library_urn="urn:adsk.eagle:library:371" deviceset="+3V3" device=""/>
-<part name="IC1" library="mcp6004-e_p" deviceset="MCP6004-E_P" device=""/>
+<part name="OPAMP1" library="mcp6004-e_p" deviceset="MCP6004-E_P" device=""/>
 <part name="GND21" library="supply1" library_urn="urn:adsk.eagle:library:371" deviceset="GND" device=""/>
 <part name="GND22" library="supply1" library_urn="urn:adsk.eagle:library:371" deviceset="GND" device=""/>
@@
 <part name="R12" library="MusicThingModular" deviceset="RESISTOR" device="7MM" value="100k"/>
 <part name="GND18" library="supply1" library_urn="urn:adsk.eagle:library:371" deviceset="GND" device=""/>
+<part name="GND19" library="supply1" library_urn="urn:adsk.eagle:library:371" deviceset="GND" device=""/>
+<part name="+3V3" library="supply1" library_urn="urn:adsk.eagle:library:371" deviceset="+3V3" device=""/>
+<part name="U$4" library="Adafruit Trellis" deviceset="NEOTRELLISKAIMAT2" device=""/>
 </parts>
 <sheets>
@@
 <attribute name="VALUE" x="23.495" y="-34.29" size="1.778" layer="96"/>
 </instance>
-<instance part="JP1" gate="A" x="-59.69" y="35.56" smashed="yes">
-<attribute name="NAME" x="-66.04" y="43.815" size="1.778" layer="95"/>
-<attribute name="VALUE" x="-66.04" y="25.4" size="1.778" layer="96"/>
-</instance>
 <instance part="ENC2" gate="G$1" x="17.78" y="-86.36" smashed="yes" rot="R270">
 <attribute name="PART" x="17.78" y="-82.55" size="1.27" layer="95"/>
@@
 <attribute name="VALUE" x="-10.16" y="12.7" size="1.778" layer="96"/>
 </instance>
-<instance part="IC1" gate="G$1" x="116.84" y="-53.34" smashed="yes">
+<instance part="OPAMP1" gate="G$1" x="116.84" y="-53.34" smashed="yes">
 <attribute name="NAME" x="116.84" y="-48.514" size="1.778" layer="95" align="center-left"/>
 <attribute name="VALUE" x="123.19" y="-48.26" size="1.778" layer="96" align="center-left"/>
@@
 <attribute name="VALUE" x="160.02" y="-30.48" size="1.778" layer="96" rot="R180"/>
 </instance>
+<instance part="GND19" gate="1" x="-48.26" y="35.56" smashed="yes" rot="R90">
+<attribute name="VALUE" x="-48.26" y="35.56" size="1.778" layer="96"/>
+</instance>
+<instance part="+3V3" gate="G$1" x="-43.18" y="33.02" smashed="yes" rot="R270">
+<attribute name="VALUE" x="-43.18" y="33.02" size="1.778" layer="96"/>
+</instance>
+<instance part="U$4" gate="G$1" x="-66.04" y="27.94" smashed="yes"/>
 </instances>
 <busses>
@@
 </segment>
 <segment>
-<pinref part="IC1" gate="G$1" pin="VSS"/>
+<pinref part="OPAMP1" gate="G$1" pin="VSS"/>
 <wire x1="154.94" y1="-60.96" x2="147.32" y2="-60.96" width="0.1524" layer="91"/>
 <pinref part="GND14" gate="1" pin="GND"/>
@@
 <pinref part="GND18" gate="1" pin="GND"/>
 <wire x1="157.48" y1="-38.1" x2="157.48" y2="-35.56" width="0.1524" layer="91"/>
+</segment>
+<segment>
+<pinref part="GND19" gate="1" pin="GND"/>
+<wire x1="-53.34" y1="35.56" x2="-50.8" y2="35.56" width="0.1524" layer="91"/>
+<pinref part="U$4" gate="G$1" pin="GND"/>
 </segment>
 </net>
@@
 </segment>
 <segment>
-<pinref part="IC1" gate="G$1" pin="VDD"/>
+<pinref part="OPAMP1" gate="G$1" pin="VDD"/>
 <wire x1="116.84" y1="-60.96" x2="109.22" y2="-60.96" width="0.1524" layer="91"/>
 <pinref part="P+3" gate="1" pin="+5V"/>
@@
 <wire x1="-30.48" y1="12.7" x2="-12.7" y2="12.7" width="0.1524" layer="91"/>
 <pinref part="+3V2" gate="G$1" pin="+3V3"/>
+</segment>
+<segment>
+<pinref part="+3V3" gate="G$1" pin="+3V3"/>
+<wire x1="-53.34" y1="33.02" x2="-45.72" y2="33.02" width="0.1524" layer="91"/>
+<pinref part="U$4" gate="G$1" pin="VIN"/>
 </segment>
 </net>
@@
 <label x="-25.4" y="-45.72" size="1.778" layer="95"/>
 </segment>
+<segment>
+<wire x1="-53.34" y1="38.1" x2="-43.18" y2="38.1" width="0.1524" layer="91"/>
+<label x="-43.18" y="38.1" size="1.778" layer="95"/>
+<pinref part="U$4" gate="G$1" pin="SCL"/>
+</segment>
 </net>
 <net name="TRLSDA" class="0">
@@
 <label x="-25.4" y="-48.26" size="1.778" layer="95"/>
 </segment>
+<segment>
+<wire x1="-53.34" y1="40.64" x2="-43.18" y2="40.64" width="0.1524" layer="91"/>
+<label x="-43.18" y="40.64" size="1.778" layer="95"/>
+<pinref part="U$4" gate="G$1" pin="SDA"/>
+</segment>
 </net>
 <net name="N$4" class="0">
@@
 <pinref part="R6" gate="G$1" pin="2"/>
 <wire x1="101.6" y1="-68.58" x2="106.68" y2="-68.58" width="0.1524" layer="91"/>
-<pinref part="IC1" gate="G$1" pin="VOUTB"/>
-<pinref part="IC1" gate="G$1" pin="VINB-"/>
+<pinref part="OPAMP1" gate="G$1" pin="VOUTB"/>
+<pinref part="OPAMP1" gate="G$1" pin="VINB-"/>
 <wire x1="106.68" y1="-68.58" x2="111.76" y2="-68.58" width="0.1524" layer="91"/>
 <wire x1="111.76" y1="-68.58" x2="116.84" y2="-68.58" width="0.1524" layer="91"/>
@@
 <net name="N$12" class="0">
 <segment>
-<pinref part="IC1" gate="G$1" pin="VOUTD"/>
+<pinref part="OPAMP1" gate="G$1" pin="VOUTD"/>
 <pinref part="R8" gate="G$1" pin="1"/>
 <wire x1="147.32" y1="-53.34" x2="152.4" y2="-53.34" width="0.1524" layer="91"/>
-<pinref part="IC1" gate="G$1" pin="VIND-"/>
+<pinref part="OPAMP1" gate="G$1" pin="VIND-"/>
 <wire x1="152.4" y1="-53.34" x2="157.48" y2="-53.34" width="0.1524" layer="91"/>
 <wire x1="157.48" y1="-53.34" x2="162.56" y2="-53.34" width="0.1524" layer="91"/>
@@
 <net name="N$13" class="0">
 <segment>
-<pinref part="IC1" gate="G$1" pin="VOUTC"/>
+<pinref part="OPAMP1" gate="G$1" pin="VOUTC"/>
 <pinref part="R7" gate="G$1" pin="1"/>
 <wire x1="147.32" y1="-68.58" x2="152.4" y2="-68.58" width="0.1524" layer="91"/>
-<pinref part="IC1" gate="G$1" pin="VINC-"/>
+<pinref part="OPAMP1" gate="G$1" pin="VINC-"/>
 <wire x1="152.4" y1="-68.58" x2="157.48" y2="-68.58" width="0.1524" layer="91"/>
 <wire x1="157.48" y1="-68.58" x2="162.56" y2="-68.58" width="0.1524" layer="91"/>
@@
 <net name="N$14" class="0">
 <segment>
-<pinref part="IC1" gate="G$1" pin="VINA+"/>
+<pinref part="OPAMP1" gate="G$1" pin="VINA+"/>
 <pinref part="R1" gate="G$1" pin="1"/>
 <wire x1="58.42" y1="-58.42" x2="116.84" y2="-58.42" width="0.1524" layer="91"/>
@@
 <net name="N$18" class="0">
 <segment>
-<pinref part="IC1" gate="G$1" pin="VINA-"/>
+<pinref part="OPAMP1" gate="G$1" pin="VINA-"/>
 <wire x1="111.76" y1="-55.88" x2="116.84" y2="-55.88" width="0.1524" layer="91"/>
 <pinref part="R5" gate="G$1" pin="2"/>
-<pinref part="IC1" gate="G$1" pin="VOUTA"/>
+<pinref part="OPAMP1" gate="G$1" pin="VOUTA"/>
 <wire x1="101.6" y1="-53.34" x2="106.68" y2="-53.34" width="0.1524" layer="91"/>
 <wire x1="106.68" y1="-53.34" x2="111.76" y2="-53.34" width="0.1524" layer="91"/>
@@
 <net name="N$11" class="0">
 <segment>
-<pinref part="IC1" gate="G$1" pin="VINB+"/>
+<pinref part="OPAMP1" gate="G$1" pin="VINB+"/>
 <wire x1="116.84" y1="-63.5" x2="58.42" y2="-63.5" width="0.1524" layer="91"/>
 <pinref part="R2" gate="G$1" pin="1"/>
@@
 <net name="N$15" class="0">
 <segment>
-<pinref part="IC1" gate="G$1" pin="VINC+"/>
+<pinref part="OPAMP1" gate="G$1" pin="VINC+"/>
 <wire x1="147.32" y1="-63.5" x2="190.5" y2="-63.5" width="0.1524" layer="91"/>
 <pinref part="R3" gate="G$1" pin="1"/>
@@
 <pinref part="R4" gate="G$1" pin="1"/>
 <wire x1="190.5" y1="-55.88" x2="190.5" y2="-58.42" width="0.1524" layer="91"/>
-<pinref part="IC1" gate="G$1" pin="VIND+"/>
+<pinref part="OPAMP1" gate="G$1" pin="VIND+"/>
 <wire x1="190.5" y1="-58.42" x2="147.32" y2="-58.42" width="0.1524" layer="91"/>
 </segment>
@@
 packages will not be understood (or retained) with this version.
 </note>
+<note version="8.5" severity="warning">
+Since Version 8.5, EAGLE supports locking for holes, vias, wires and polygons.
+The locking property on all objects of these types will not be understood in this version.
+</note>
 </compatibility>

Commit message: improved circuit and pcb£
Parts:
- added R13, R14, R15: 100k, MusicThingModular:RESISTOR7MM
- added U$5: DAC8568C, analog-devices-3:DAC8568C
- added X1: OPAMP, ngspice-simulation:OPAMP
Connections:
- removed net N$2: D1.C, U$2.IN
- new net DACOUTCV1: U$5.VOUTA, X1.P
- new net DACOUTCV2: U$5.VOUTB
- new net DACOUTCV3: U$5.VOUTC
- new net DACOUTCV4: U$5.VOUTD
- new net DACOUTTR1: U$5.VOUTE
- new net DACOUTTR2: U$5.VOUTF
- new net DACOUTTR3: U$5.VOUTG
- new net DACOUTTR4: U$5.VOUTH
- new net N$10: R14.2, R15.1, X1.N
- new net N$7: CV1.TIP, R13.2
- new net N$8: R13.1, R15.2, X1.VOUT
- new net VCC: D1.C, U$2.IN, X1.VDD
- net +5V: now also U$5.AVDD
- net CVIN1: now also R10.1
- net CVIN2: now also R9.1
- net CVIN3: now also R11.1
- net CVIN4: now also R12.1
- net DACCLR: now also U$5.CLR
- net DACDATA: now also U$5.DIN
- net DACLDAC: now also U$5.LDAC
- net DACSPICLK: now also U$5.SCLK
- net DACSS: now also U$5.SYNC
- net GND: now also R14.1, U$5.GND, X1.VSS; no longer CV1.SWITCH, CV2.SWITCH, CV3.SWITCH, CV4.SWITCH, TR1.SWITCH, TR2.SWITCH, TR3.SWITCH, TR4.SWITCH
- net N$12: no longer R12.1
- net N$13: no longer R11.1
- net N$18: no longer R10.1
- net N$4: no longer R9.1
Other:
- moved on the sheet: CV1, CV2, CV3, CV4, D1, ENC1, ENC2, IN1, IN2, IN3, IN4, OPAMP1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

Commit message: updated circuit and pcb
Other:
- moved on the sheet: CV1, D1, R13, R14, R15, SV1, U$2, X1

Commit message: updated circuit and pcb
Parts:
- added OPAMP2: MCP6004-E_P, mcp6004-e_p:MCP6004-E_P
- added R16, R17, R18, R19, R20, R21, R22, R23, R24, R25, R26, R27: 100k, MusicThingModular:RESISTOR7MM
Connections:
- new net N$17: OPAMP2.VINB-, R16.2, R17.1
- new net N$19: CV2.TIP, R18.2
- new net N$2: OPAMP2.VOUTB, R17.2, R18.1
- new net N$20: CV3.TIP, R21.2
- new net N$21: OPAMP2.VOUTC, R19.1, R21.1
- new net N$22: OPAMP2.VINC-, R19.2, R20.1
- new net N$23: OPAMP2.VINA-, R22.2, R23.1
- new net N$24: OPAMP2.VOUTA, R23.2, R24.1
- new net N$25: CV1.TIP, R24.2
- new net N$26: OPAMP2.VIND-, R25.1, R26.2
- new net N$27: OPAMP2.VOUTD, R26.1, R27.1
- new net N$28: CV4.TIP, R27.2
- net DACOUTCV1: now also OPAMP2.VINA+; no longer X1.P
- net DACOUTCV2: now also OPAMP2.VINB+
- net DACOUTCV3: now also OPAMP2.VINC+
- net DACOUTCV4: now also OPAMP2.VIND+
- net DACOUTTR1: now also X1.P
- net GND: now also OPAMP2.VSS, R16.1, R20.2, R22.1, R25.2
- net N$7: now also TR1.TIP; no longer CV1.TIP
- net VCC: now also OPAMP2.VDD
Other:
- moved on the sheet: CV1, CV2, CV3, CV4, R13, R14, R15, TR1, X1

Commit message: updated circuit and pcb
Parts:
- removed OPAMP2: MCP6004-E_P, mcp6004-e_p:MCP6004-E_P
- added IC1, IC2: TL074CN, TL074CN:TL074CN
Connections:
- net DACOUTCV1: now also IC1.1IN+; no longer OPAMP2.VINA+
- net DACOUTCV2: now also IC1.2IN+; no longer OPAMP2.VINB+
- net DACOUTCV3: now also IC1.3IN+; no longer OPAMP2.VINC+
- net DACOUTCV4: now also IC1.4IN+; no longer OPAMP2.VIND+
- net GND: now also IC1.VCC-; no longer OPAMP2.VSS
- net N$17: now also IC1.2IN-; no longer OPAMP2.VINB-
- net N$2: now also IC1.2OUT; no longer OPAMP2.VOUTB
- net N$21: now also IC1.3OUT; no longer OPAMP2.VOUTC
- net N$22: now also IC1.3IN-; no longer OPAMP2.VINC-
- net N$23: now also IC1.1IN-; no longer OPAMP2.VINA-
- net N$24: now also IC1.1OUT; no longer OPAMP2.VOUTA
- net N$26: now also IC1.4IN-; no longer OPAMP2.VIND-
- net N$27: now also IC1.4OUT; no longer OPAMP2.VOUTD
- net VCC: now also IC1.VCC+; no longer OPAMP2.VDD
Other:
- moved on the sheet: CV1, CV2, CV3, CV4, R13, R14, R15, R16, R17, R18, R19, R20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

Commit message: finished schematic
Parts:
- removed R13, R14, R15: 100k, MusicThingModular:RESISTOR7MM
- removed X1: OPAMP, ngspice-simulation:OPAMP
- added D2: 1N4004, diode:1N4004
- added R28, R29, R30, R31, R32, R33, R34, R35, R36, R37, R38, R39: 100k, MusicThingModular:RESISTOR7MM
Connections:
- removed net N$10: R14.2, R15.1, X1.N
- removed net N$8: R13.1, R15.2, X1.VOUT
- new net N$29: D2.C, SV1.1, SV1.2
- new net N$30: IC2.1IN-, R28.2, R29.1
- new net N$31: IC2.1OUT, R29.2, R30.1
- new net N$32: IC2.2IN-, R31.2, R32.1
- new net N$33: R30.2, TR1.TIP
- new net N$34: R33.2, TR2.TIP
- new net N$35: IC2.3IN-, R34.2, R35.1
- new net N$36: R36.2, TR3.TIP
- new net N$37: IC2.3OUT, R34.1, R36.1
- new net N$38: IC2.4IN-, R37.1, R38.2
- new net N$39: IC2.4OUT, R38.1, R39.1
- new net N$40: R39.2, TR4.TIP
- new net VSS: D2.A, IC1.VCC-, IC2.VCC-
- net DACOUTTR1: now also IC2.1IN+; no longer X1.P
- net DACOUTTR2: now also IC2.2IN+
- net DACOUTTR3: now also IC2.3IN+
- net DACOUTTR4: now also IC2.4IN+
- net GND: now also R28.1, R31.1, R35.2, R37.2; no longer IC1.VCC-, R14.1, X1.VSS
- net N$7: now also IC2.2OUT, R32.2, R33.1; no longer R13.2, TR1.TIP
- net VCC: now also IC2.VCC+; no longer X1.VDD
Other:
- moved on the sheet: CV1, CV2, CV3, CV4, D1, IC1, IC2, R16, R17, R18, R19, R20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

Commit message: better pcb
Connections:
- net DACOUTCV2: now also U$5.VOUTC; no longer U$5.VOUTB
- net DACOUTCV3: now also U$5.VOUTE; no longer U$5.VOUTC
- net DACOUTCV4: now also U$5.VOUTG; no longer U$5.VOUTD
- net DACOUTTR1: now also U$5.VOUTB; no longer U$5.VOUTE
- net DACOUTTR2: now also U$5.VOUTD; no longer U$5.VOUTF
- net DACOUTTR3: now also U$5.VOUTF; no longer U$5.VOUTG
Other:
- moved on the sheet: ENC1, ENC2, S1, S2

Commit message: better pcb
Parts:
- removed R37, R38, R39: 100k, MusicThingModular:RESISTOR7MM
- added R13, R14, R15: 100k, Clean-Kong:R-EU_R0805
- R1, R10, R11, R12, R16, R17, R18, R19, R2, R20, R21, R22, R23, R24, R25, R26, R27, R28, R29, R3, R30, R31, R32, R33, R34, R35, R36, R4, R5, R6, R7, R8, R9: device MusicThingModular:RESISTOR7MM -> Clean-Kong:R-EU_R0805
- renumbered U$5 to DAC8568C
Connections:
- net CVIN2: now also R9.2; no longer R9.1
- net CVIN3: now also R11.2; no longer R11.1
- net ENC1PINA: now also U$1.15/A1; no longer U$1.1/TX
- net ENC1PINB: now also U$1.16/A2; no longer U$1.2
- net ENC1SW: now also U$1.14/A0; no longer U$1.0/RX
- net ENC2PINA: now also U$1.1/TX; no longer U$1.15/A1
- net ENC2PINB: now also U$1.2; no longer U$1.16/A2
- net ENC2SW: now also U$1.0/RX; no longer U$1.14/A0
- net GND: now also R11.1, R34.2, R9.1; no longer R11.2, R37.2, R9.2
- net N$11: now also R2.2; no longer R2.1
- net N$15: now also R3.2; no longer R3.1
- net N$31: now also R13.1; no longer R30.1
- net N$33: now also R13.2; no longer R30.2
- net N$34: now also R14.2; no longer R33.2
- net N$35: now also R33.2, R34.1; no longer R34.2, R35.1
- net N$36: now also R30.2; no longer R36.2
- net N$37: now also R30.1, R33.1; no longer R34.1, R36.1
- net N$38: now also R35.1, R36.2; no longer R37.1, R38.2
- net N$39: now also R15.1, R36.1; no longer R38.1, R39.1
- net N$40: now also R15.2; no longer R39.2
- net N$5: now also R2.1; no longer R2.2
- net N$6: now also R3.1; no longer R3.2
- net N$7: now also R14.1; no longer R33.1
Other:
- moved on the sheet: R11, R2, R3, R30, R33, R34, R35, R36, R9
