File: Schematic/Eagle/KaiMat/kaimat.sch (EAGLE design)
At the start: 63 parts, among them IC1 TL074CN, IC2 TL074CN

Commit message: better pcb
Parts:
- renumbered IC1 to TL04CN-2, IC2 to TL04CN-1, OPAMP1 to MCP6004-E_P, U$3 to SSD1306-128X64
