File: Schematic/Eagle/KaiMat/kaimat.brd (EAGLE design)
At the start: 60.1 x 110.5 mm, 35 parts, among them IC1 MCP6004-E_P

Commit message: improved schematic
Parts:
- removed IC1: MCP6004-E_P, mcp6004-e_p:DIP781W56P254L1918H533Q14N
- removed JP1: (no value), microbuilder:5P_EDGECONNECT
- added OPAMP1: MCP6004-E_P, mcp6004-e_p:DIP781W56P254L1918H533Q14N
- added U$4: NEOTRELLISKAIMAT2, Adafruit Trellis:NEOTRELLISKAIMAT2
- moved U$1 2.74 mm to (18.5, 30.8)
- moved U$2 1.00 mm to (34.9, 12.6)
- moved ENC1 0.50 mm to (35.2, 75.7)
- moved ENC2 0.50 mm to (50.8, 75.7)
- moved S1 0.50 mm to (35.2, 63.5)
- moved S2 0.50 mm to (50.8, 63.5)
Connections:
- net +3V3: now also U$4.VIN
- net +5V: now also OPAMP1.4; no longer IC1.4
- net GND: now also OPAMP1.11, U$4.GND; no longer IC1.11
- net N$11: now also OPAMP1.5; no longer IC1.5
- net N$12: now also OPAMP1.13, OPAMP1.14; no longer IC1.13, IC1.14
- net N$13: now also OPAMP1.8, OPAMP1.9; no longer IC1.8, IC1.9
- net N$14: now also OPAMP1.3; no longer IC1.3
- net N$15: now also OPAMP1.10; no longer IC1.10
- net N$16: now also OPAMP1.12; no longer IC1.12
- net N$18: now also OPAMP1.1, OPAMP1.2; no longer IC1.1, IC1.2
- net N$4: now also OPAMP1.6, OPAMP1.7; no longer IC1.6, IC1.7
- net TRLSCL: now also U$4.SCL
- net TRLSDA: now also U$4.SDA
Routing:
- net GND: track 365.5 -> 358.2 mm
- net +5V: track 8.19 -> 6.51 mm
- net N$2: track 7.00 -> 6.00 mm
Other:
- board size 60.1 x 110.5 mm -> 60 x 110.5 mm

Commit message: improved schematic
Parts:
- moved D1 0.50 mm to (43.0, 9.53)
- moved OPAMP1 0.50 mm to (36.0, 33.5)
- moved U$2 0.50 mm to (34.4, 12.6)
Routing:
- net GND: track 358.2 -> 387.7 mm
- net N$2: track 6.00 -> 7.00 mm
- net N$1: track 8.48 -> 7.98 mm
- net +5V: track 6.51 -> 6.01 mm

Commit message: improved circuit and pcb£
Parts:
- added R13, R14, R15: 100k, MusicThingModular:7MM_RESISTOR
- added U$5: DAC8568C, analog-devices-3:TSSOP16
Connections:
- net N$2 renamed VCC
- new net DACOUTCV1: U$5.4
- new net DACOUTCV2: U$5.13
- new net DACOUTCV3: U$5.5
- new net DACOUTCV4: U$5.12
- new net DACOUTTR1: U$5.6
- new net DACOUTTR2: U$5.11
- new net DACOUTTR3: U$5.7
- new net DACOUTTR4: U$5.10
- new net N$10: R14.2, R15.1
- new net N$7: CV1.P$1_TIP, R13.2
- new net N$8: R13.1, R15.2
- net +5V: now also U$5.3
- net CVIN1: now also R10.1
- net CVIN2: now also R9.1
- net CVIN3: now also R11.1
- net CVIN4: now also R12.1
- net DACCLR: now also U$5.9
- net DACDATA: now also U$5.15
- net DACLDAC: now also U$5.1
- net DACSPICLK: now also U$5.16
- net DACSS: now also U$5.2
- net GND: now also R14.1, U$5.14; no longer CV1.P$2_SWITCH, CV2.P$2_SWITCH, CV3.P$2_SWITCH, CV4.P$2_SWITCH, TR1.P$2_SWITCH, TR2.P$2_SWITCH, TR3.P$2_SWITCH, TR4.P$2_SWITCH
- net N$12: no longer R12.1
- net N$13: no longer R11.1
- net N$18: no longer R10.1
- net N$4: no longer R9.1
Routing:
- net GND: track 387.7 -> 363.7 mm

Commit message: updated circuit and pcb
Parts:
- flipped U$5 to the bottom
Changed lines of the file:
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@@
 </element>
 <element name="U$4" library="Adafruit Trellis" package="NEOTRELLISKAIMAT2" value="NEOTRELLISKAIMAT2" x="0" y="60" smashed="yes"/>
-<element name="U$5" library="analog-devices-3" package="TSSOP16" value="DAC8568C" x="34" y="49.5" smashed="yes">
-<attribute name="NAME" x="31.825" y="52.675" size="1.27" layer="25"/>
-<attribute name="VALUE" x="30.825" y="45.055" size="1.27" layer="27"/>
+<element name="U$5" library="analog-devices-3" package="TSSOP16" value="DAC8568C" x="34" y="49.5" smashed="yes" rot="MR0">
+<attribute name="NAME" x="36.175" y="52.675" size="1.27" layer="26" rot="MR0"/>
+<attribute name="VALUE" x="37.175" y="45.055" size="1.27" layer="28" rot="MR0"/>
 </element>
 <element name="R13" library="MusicThingModular" package="7MM_RESISTOR" value="100k" x="4" y="-44" smashed="yes">
@@
 <wire x1="25.019" y1="97.005" x2="14.986" y2="97.005" width="0" layer="19" extent="1-1"/>
 <wire x1="25.019" y1="97.0002" x2="25.019" y2="97.005" width="0" layer="19" extent="1-1"/>
-<wire x1="36.875" y1="50.475" x2="35.235" y2="65.7876" width="0" layer="19" extent="1-16"/>
-<wire x1="39.905" y1="33.5" x2="36.875" y2="50.475" width="0" layer="19" extent="1-1"/>
+<wire x1="31.125" y1="50.475" x2="35.235" y2="65.7876" width="0" layer="19" extent="1-16"/>
+<wire x1="39.905" y1="33.5" x2="31.125" y2="50.475" width="0" layer="19" extent="1-1"/>
 <wire x1="8.81" y1="-30" x2="12.467" y2="1.27" width="0" layer="19" extent="16-16"/>
 <wire x1="8.81" y1="-33.5" x2="8.81" y2="-30" width="0" layer="19" extent="1-1"/>
@@
 <contactref element="OPAMP1" pad="4"/>
 <contactref element="U$5" pad="3"/>
-<wire x1="32.095" y1="33.5" x2="31.125" y2="50.475" width="0" layer="19" extent="1-1"/>
+<wire x1="32.095" y1="33.5" x2="36.875" y2="50.475" width="0" layer="19" extent="1-1"/>
 <wire x1="32.012" y1="2.9704" x2="32.095" y2="33.5" width="0" layer="19" extent="1-1"/>
 </signal>
@@
 <contactref element="U$1" pad="7"/>
 <contactref element="U$5" pad="9"/>
-<wire x1="10.876" y1="23.181" x2="36.875" y2="47.225" width="0" layer="19" extent="1-1"/>
+<wire x1="10.876" y1="23.181" x2="31.125" y2="47.225" width="0" layer="19" extent="1-1"/>
 </signal>
 <signal name="DACLDAC">
 <contactref element="U$1" pad="6"/>
 <contactref element="U$5" pad="1"/>
-<wire x1="10.876" y1="20.641" x2="31.125" y2="51.775" width="0" layer="19" extent="1-1"/>
+<wire x1="10.876" y1="20.641" x2="36.875" y2="51.775" width="0" layer="19" extent="1-1"/>
 </signal>
 <signal name="DACSS">
 <contactref element="U$1" pad="5"/>
 <contactref element="U$5" pad="2"/>
-<wire x1="10.876" y1="18.101" x2="31.125" y2="51.125" width="0" layer="19" extent="1-1"/>
+<wire x1="10.876" y1="18.101" x2="36.875" y2="51.125" width="0" layer="19" extent="1-1"/>
 </signal>
 <signal name="DACSPICLK">
 <contactref element="U$1" pad="4/CANRX"/>
 <contactref element="U$5" pad="16"/>
-<wire x1="10.876" y1="15.561" x2="36.875" y2="51.775" width="0" layer="19" extent="1-1"/>
+<wire x1="10.876" y1="15.561" x2="31.125" y2="51.775" width="0" layer="19" extent="1-1"/>
 </signal>
 <signal name="DACDATA">
 <contactref element="U$1" pad="3/CANTX"/>
 <contactref element="U$5" pad="15"/>
-<wire x1="10.876" y1="13.021" x2="36.875" y2="51.125" width="0" layer="19" extent="1-1"/>
+<wire x1="10.876" y1="13.021" x2="31.125" y2="51.125" width="0" layer="19" extent="1-1"/>
 </signal>
 <signal name="CVIN1">

Commit message: updated circuit and pcb
Parts:
- added OPAMP2: MCP6004-E_P, mcp6004-e_p:DIP781W56P254L1918H533Q14N
- added R16, R17, R18, R19, R20, R21, R22, R23, R24, R25, R26, R27: 100k, MusicThingModular:7MM_RESISTOR
- moved U$5 21.0 mm to (34.0, 28.5)
- moved OPAMP1 16.7 mm to (49.0, 23.0), turned to 90 degrees
- moved ENC2 0.25 mm to (51.1, 75.7)
- moved S2 0.25 mm to (51.1, 63.5)
Connections:
- new net N$17: OPAMP2.6, R16.2, R17.1
- new net N$19: CV2.P$1_TIP, R18.2
- new net N$2: OPAMP2.7, R17.2, R18.1
- new net N$20: CV3.P$1_TIP, R21.2
- new net N$21: OPAMP2.8, R19.1, R21.1
- new net N$22: OPAMP2.9, R19.2, R20.1
- new net N$23: OPAMP2.2, R22.2, R23.1
- new net N$24: OPAMP2.1, R23.2, R24.1
- new net N$25: CV1.P$1_TIP, R24.2
- new net N$26: OPAMP2.13, R25.1, R26.2
- new net N$27: OPAMP2.14, R26.1, R27.1
- new net N$28: CV4.P$1_TIP, R27.2
- net DACOUTCV1: now also OPAMP2.3
- net DACOUTCV2: now also OPAMP2.5
- net DACOUTCV3: now also OPAMP2.10
- net DACOUTCV4: now also OPAMP2.12
- net GND: now also OPAMP2.11, R16.1, R20.2, R22.1, R25.2
- net N$7: now also TR1.P$1_TIP; no longer CV1.P$1_TIP
- net VCC: now also OPAMP2.4

Commit message: updated circuit and pcb
Parts:
- removed OPAMP2: MCP6004-E_P, mcp6004-e_p:DIP781W56P254L1918H533Q14N
- added IC1, IC2: TL074CN, TL074CN:DIP794W53P254L1930H508Q14N
- moved U$5 1.12 mm to (33.0, 28.0), flipped to the top
Connections:
- new net VCC+: IC2.4
- new net VCC-: IC2.11
- net DACOUTCV1: now also IC1.3; no longer OPAMP2.3
- net DACOUTCV2: now also IC1.5; no longer OPAMP2.5
- net DACOUTCV3: now also IC1.10; no longer OPAMP2.10
- net DACOUTCV4: now also IC1.12; no longer OPAMP2.12
- net GND: now also IC1.11; no longer OPAMP2.11
- net N$17: now also IC1.6; no longer OPAMP2.6
- net N$2: now also IC1.7; no longer OPAMP2.7
- net N$21: now also IC1.8; no longer OPAMP2.8
- net N$22: now also IC1.9; no longer OPAMP2.9
- net N$23: now also IC1.2; no longer OPAMP2.2
- net N$24: now also IC1.1; no longer OPAMP2.1
- net N$26: now also IC1.13; no longer OPAMP2.13
- net N$27: now also IC1.14; no longer OPAMP2.14
- net VCC: now also IC1.4; no longer OPAMP2.4
Routing:
- net +3V3: track 0.00 -> 110.3 mm
- net GND: track 363.7 -> 392.0 mm

Commit message: updated circuit and pcb
Parts:
- moved IC2 1.58 mm to (45.5, 50.0)
- moved IC1 0.50 mm to (45.5, 37.5)

Commit message: finished schematic
Parts:
- removed R13, R14, R15: 100k, MusicThingModular:7MM_RESISTOR
- added D2: 1N4004, diode:DO41-10
- added R28, R29, R30, R31, R32, R33, R34, R35, R36, R37, R38, R39: 100k, MusicThingModular:7MM_RESISTOR
- moved IC2 4.03 mm to (49.0, 52.0)
- moved IC1 3.50 mm to (49.0, 37.5)
- moved U$5 1.41 mm to (34.0, 27.0)
Connections:
- removed net N$10: R14.2, R15.1
- removed net N$8: R13.1, R15.2
- removed net VCC+: IC2.4
- removed net VCC-: IC2.11
- new net N$29: D2.C, SV1.1, SV1.2
- new net N$30: IC2.2, R28.2, R29.1
- new net N$31: IC2.1, R29.2, R30.1
- new net N$32: IC2.6, R31.2, R32.1
- new net N$33: R30.2, TR1.P$1_TIP
- new net N$34: R33.2, TR2.P$1_TIP
- new net N$35: IC2.9, R34.2, R35.1
- new net N$36: R36.2, TR3.P$1_TIP
- new net N$37: IC2.8, R34.1, R36.1
- new net N$38: IC2.13, R37.1, R38.2
- new net N$39: IC2.14, R38.1, R39.1
- new net N$40: R39.2, TR4.P$1_TIP
- new net VSS: D2.A, IC1.11, IC2.11
- net DACOUTTR1: now also IC2.3
- net DACOUTTR2: now also IC2.5
- net DACOUTTR3: now also IC2.10
- net DACOUTTR4: now also IC2.12
- net GND: now also R28.1, R31.1, R35.2, R37.2; no longer IC1.11, R14.1
- net N$7: now also IC2.7, R32.2, R33.1; no longer R13.2, TR1.P$1_TIP
- net VCC: now also IC2.4
Routing:
- net GND: track 392.0 -> 371.0 mm
- net N$1: track 7.98 -> 5.44 mm
