File: HardWare/Board/SPosition.brd (EAGLE design)
At the start: 60 x 110 mm, 72 parts

Commit message: pcb rev5
Routing:
- net VSS: track 83.0 -> 82.3 mm
- net N$22: track 22.3 -> 21.7 mm
Changed lines of the file:
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@@
 <drawing>
 <settings>
-<setting alwaysvectorfont="no"/>
+<setting alwaysvectorfont="yes"/>
 <setting verticaltext="up"/>
 </settings>
@@
 <contactref element="R19" pad="2"/>
 <wire x1="54.5" y1="36.45" x2="54.575" y2="36.425" width="0.1524" layer="16"/>
-<wire x1="54.575" y1="35.925" x2="55.57" y2="36.92" width="0.1524" layer="16"/>
-<wire x1="55.57" y1="36.92" x2="56.86" y2="36.92" width="0.1524" layer="16"/>
+<wire x1="56.86" y1="36.92" x2="54.97" y2="36.92" width="0.1524" layer="16"/>
+<wire x1="54.5" y1="36.45" x2="54.97" y2="36.92" width="0.1524" layer="16"/>
 <wire x1="53.5" y1="55.05" x2="53.5" y2="41" width="0.1524" layer="16"/>
 <wire x1="53.5" y1="41" x2="54.575" y2="39.925" width="0.1524" layer="16"/>
 <wire x1="54.575" y1="39.925" x2="54.575" y2="36.425" width="0.1524" layer="16"/>
-<wire x1="54.575" y1="36.425" x2="54.575" y2="35.925" width="0.1524" layer="16"/>
 </signal>
 <signal name="N$20">
@@
 <contactref element="R21" pad="1"/>
 <contactref element="R19" pad="1"/>
-<wire x1="56.86" y1="34.38" x2="56.59" y2="34.65" width="0.1524" layer="16"/>
-<wire x1="56.59" y1="34.65" x2="54.5" y2="34.55" width="0.1524" layer="16"/>
 <wire x1="51" y1="84.25" x2="46.75" y2="88.5" width="0.1524" layer="16"/>
 <wire x1="46.75" y1="88.55" x2="46.75" y2="88.5" width="0.1524" layer="16"/>
@@
 <wire x1="52.5" y1="38.74" x2="56.86" y2="34.38" width="0.1524" layer="1"/>
 <wire x1="52.5" y1="70.5" x2="52.5" y2="38.74" width="0.1524" layer="1"/>
+<wire x1="56.86" y1="34.38" x2="54.67" y2="34.38" width="0.1524" layer="16"/>
+<wire x1="54.67" y1="34.38" x2="54.5" y2="34.55" width="0.1524" layer="16"/>
 </signal>
 <signal name="N$23">
@@
 <contactref element="C7-100N" pad="1"/>
 <contactref element="C8-100N" pad="1"/>
-<wire x1="52.3" y1="2.75" x2="49.33" y2="2.75" width="0.1524" layer="16"/>
-<wire x1="49.33" y1="2.75" x2="48.58" y2="3.5" width="0.1524" layer="16"/>
+<wire x1="52.3" y1="2.75" x2="50.08" y2="2.75" width="0.1524" layer="16"/>
+<wire x1="50.08" y1="2.75" x2="49.33" y2="3.5" width="0.1524" layer="16"/>
 <wire x1="52.3" y1="5.75" x2="52.2575" y2="5.7075" width="0.1524" layer="16"/>
-<wire x1="52.2575" y1="5.7075" x2="50.7875" y2="5.7075" width="0.1524" layer="16"/>
-<wire x1="50.7875" y1="5.7075" x2="48.58" y2="3.5" width="0.1524" layer="16"/>
+<wire x1="52.2575" y1="5.7075" x2="51.5375" y2="5.7075" width="0.1524" layer="16"/>
+<wire x1="51.5375" y1="5.7075" x2="49.33" y2="3.5" width="0.1524" layer="16"/>
+<wire x1="49.33" y1="3.5" x2="48.58" y2="3.5" width="0.1524" layer="16"/>
 </signal>
 <signal name="N$29">

Commit message: pcb rev5
Parts:
- moved C4-100N 0.75 mm to (25.5, 16.5)
- moved MCP4922-1 0.50 mm to (46.0, 8.00)
- moved MCP4922-2 0.50 mm to (56.5, 8.00)
- moved C3-100N 0.25 mm to (22.5, 16.5)
- moved C7-100N 0.25 mm to (53.2, 3.00)
- moved C8-100N 0.25 mm to (53.2, 6.00)
Routing:
- net DAC2SCK: track 28.4 -> 29.0 mm
- net DAC1CS: track 5.54 -> 6.06 mm
- net DAC1SCK: track 5.54 -> 6.04 mm
- net DAC1MOSI: track 5.54 -> 6.04 mm
- net GND: track 604.1 -> 603.6 mm
- net DAC2CS: track 27.4 -> 27.9 mm
- net DAC1LDAC: track 14.1 -> 14.6 mm
- net CV4: track 31.4 -> 31.9 mm
- net CV3: track 25.9 -> 26.4 mm
- net CV2: track 27.7 -> 28.2 mm
- net CV1: track 29.3 -> 29.8 mm

Commit message: added gerber files
Parts:
- moved C4-100N 5.02 mm to (26.0, 11.5)
- moved C3-100N 5.00 mm to (22.5, 11.5)
Routing:
- net +5V: track 148.8 -> 159.3 mm
- net GND: track 603.6 -> 601.5 mm
Changed lines of the file:
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@@
 <setting verticaltext="up"/>
 </settings>
-<grid distance="0.25" unitdist="mm" unit="mm" style="lines" multiple="1" display="yes" altdistance="0.01" altunitdist="mm" altunit="mm"/>
+<grid distance="0.5" unitdist="mm" unit="mm" style="lines" multiple="1" display="yes" altdistance="0.01" altunitdist="mm" altunit="mm"/>
 <layers>
 <layer number="1" name="Top" color="4" fill="1" visible="yes" active="yes"/>
@@
 <attribute name="SPICEPREFIX" value="C" x="53.25" y="6" size="1.778" layer="28" rot="MR180" display="off"/>
 </element>
-<element name="C3-100N" library="rcl" library_urn="urn:adsk.eagle:library:334" package="C0805" package3d_urn="urn:adsk.eagle:package:23617/2" value="100n" x="22.5" y="16.5" smashed="yes" rot="MR270">
-<attribute name="NAME" x="21.611" y="17.75" size="0.6096" layer="26" font="vector" ratio="20" rot="MR270" align="bottom-center"/>
-<attribute name="SPICEPREFIX" value="C" x="22.5" y="16.5" size="1.778" layer="28" rot="MR270" display="off"/>
-</element>
-<element name="C4-100N" library="rcl" library_urn="urn:adsk.eagle:library:334" package="C0805" package3d_urn="urn:adsk.eagle:package:23617/2" value="100n" x="25.5" y="16.5" smashed="yes" rot="MR270">
-<attribute name="NAME" x="24.361" y="17.75" size="0.6096" layer="26" font="vector" ratio="20" rot="MR270" align="bottom-center"/>
-<attribute name="SPICEPREFIX" value="C" x="25.5" y="16.5" size="1.778" layer="28" rot="MR270" display="off"/>
+<element name="C3-100N" library="rcl" library_urn="urn:adsk.eagle:library:334" package="C0805" package3d_urn="urn:adsk.eagle:package:23617/2" value="100n" x="22.5" y="11.5" smashed="yes" rot="MR270">
+<attribute name="NAME" x="21.611" y="12.75" size="0.6096" layer="26" font="vector" ratio="20" rot="MR270" align="bottom-center"/>
+<attribute name="SPICEPREFIX" value="C" x="22.5" y="11.5" size="1.778" layer="28" rot="MR270" display="off"/>
+</element>
+<element name="C4-100N" library="rcl" library_urn="urn:adsk.eagle:library:334" package="C0805" package3d_urn="urn:adsk.eagle:package:23617/2" value="100n" x="26" y="11.5" smashed="yes" rot="MR270">
+<attribute name="NAME" x="24.861" y="12.75" size="0.6096" layer="26" font="vector" ratio="20" rot="MR270" align="bottom-center"/>
+<attribute name="SPICEPREFIX" value="C" x="26" y="11.5" size="1.778" layer="28" rot="MR270" display="off"/>
 </element>
 </elements>
@@
 <wire x1="21" y1="79.75" x2="22.325" y2="79.75" width="0.1524" layer="16"/>
 <wire x1="6.371" y1="11.125" x2="8.25" y2="11.125" width="0.1524" layer="16"/>
+<wire x1="8.25" y1="8.665" x2="8.25" y2="11.125" width="0.1524" layer="16"/>
 <wire x1="8.25" y1="11.125" x2="8.25" y2="13.665" width="0.1524" layer="16"/>
 <wire x1="6.371" y1="8.585" x2="6.456" y2="8.5" width="0.1524" layer="16"/>
@@
 <contactref element="C3-100N" pad="2"/>
 <contactref element="C4-100N" pad="2"/>
-<wire x1="8.25" y1="11.125" x2="22.5" y2="11.125" width="0.1524" layer="16"/>
-<wire x1="22.5" y1="11.125" x2="25.525" y2="11.125" width="0.1524" layer="16"/>
-<wire x1="25.5" y1="15.55" x2="25.525" y2="15.525" width="0.1524" layer="16"/>
-<wire x1="25.525" y1="15.525" x2="25.525" y2="11.125" width="0.1524" layer="16"/>
-<wire x1="22.5" y1="15.55" x2="22.5" y2="11.125" width="0.1524" layer="16"/>
+<wire x1="8.25" y1="8.665" x2="22.49" y2="8.665" width="0.1524" layer="16"/>
+<wire x1="22.49" y1="8.675" x2="26.025" y2="8.675" width="0.1524" layer="16"/>
+<wire x1="26" y1="10.55" x2="26.025" y2="10.525" width="0.1524" layer="16"/>
+<wire x1="26.025" y1="10.525" x2="26.025" y2="8.675" width="0.1524" layer="16"/>
+<wire x1="22.5" y1="10.55" x2="22.49" y2="10.54" width="0.1524" layer="16"/>
+<wire x1="22.49" y1="10.54" x2="22.49" y2="8.675" width="0.1524" layer="16"/>
+<wire x1="22.49" y1="8.675" x2="22.49" y2="8.665" width="0.1524" layer="16"/>
 <wire x1="4.2595125" y1="1.0922" x2="55.8114875" y2="1.0922" width="0.1524" layer="16"/>
 <wire x1="56.6433" y1="63.7004" x2="56.8437" y2="63.7004" width="0.1524" layer="16"/>
@@
 <contactref element="C3-100N" pad="1"/>
 <contactref element="C4-100N" pad="1"/>
-<wire x1="22.5" y1="17.45" x2="22.5" y2="21.29" width="0.1524" layer="16"/>
-<wire x1="25.5" y1="17.45" x2="25.5" y2="21.29" width="0.1524" layer="16"/>
-<wire x1="25.5" y1="21.29" x2="23.4508" y2="21.29" width="0.1524" layer="16"/>
+<wire x1="22.5" y1="12.45" x2="22.5" y2="21.29" width="0.1524" layer="16"/>
+<wire x1="26" y1="12.45" x2="26" y2="21.29" width="0.1524" layer="16"/>
+<wire x1="26" y1="21.29" x2="23.4508" y2="21.29" width="0.1524" layer="16"/>
 </signal>
 <signal name="+3V3">
@@
 <via x="7.5" y="78" extent="1-16" drill="0.35"/>
 <wire x1="7.5" y1="78" x2="9.5" y2="78" width="0.1524" layer="16"/>
-<wire x1="16.0928" y1="70.4072" x2="16.0928" y2="64.70388125" width="0.1524" layer="16"/>
-<wire x1="17.5" y1="63.29668125" x2="17.5" y2="53.5" width="0.1524" layer="16"/>
-<wire x1="16.0928" y1="64.70388125" x2="17.5" y2="63.29668125" width="0.1524" layer="16"/>
+<wire x1="17.5" y1="69" x2="17.5" y2="53.5" width="0.1524" layer="16"/>
 <wire x1="17.5" y1="53.5" x2="17.879" y2="53.121" width="0.1524" layer="16"/>
 <wire x1="17.879" y1="53.121" x2="19.376" y2="53.121" width="0.1524" layer="16"/>
-<wire x1="14.5" y1="72" x2="16.0928" y2="70.4072" width="0.1524" layer="16"/>
+<wire x1="14.5" y1="72" x2="17.5" y2="69" width="0.1524" layer="16"/>
 <wire x1="9.5" y1="78" x2="9.5" y2="72" width="0.1524" layer="16"/>
 <wire x1="9.5" y1="72" x2="14.5" y2="72" width="0.1524" layer="16"/>
@@
 <contactref element="U$1" pad="22/A8"/>
 <wire x1="6.235" y1="68.192" x2="6.235" y2="70" width="0.1524" layer="16"/>
-<wire x1="6.235" y1="70" x2="15" y2="70" width="0.1524" layer="16"/>
-<wire x1="16.5" y1="50.5" x2="16.5" y2="62.5" width="0.1524" layer="16"/>
-<wire x1="16.5" y1="50.5" x2="16.581" y2="50.581" width="0.1524" layer="16"/>
-<wire x1="16.581" y1="50.581" x2="19.376" y2="50.581" width="0.1524" layer="16"/>
-<wire x1="16.5" y1="62.5" x2="15" y2="64" width="0.1524" layer="16"/>
-<wire x1="15" y1="64" x2="15" y2="70" width="0.1524" layer="16"/>
+<wire x1="6.235" y1="70" x2="15.25" y2="70" width="0.1524" layer="16"/>
+<wire x1="19.376" y1="50.581" x2="17" y2="50.581" width="0.1524" layer="16"/>
+<wire x1="16.5" y1="62.5" x2="15.25" y2="63.75" width="0.1524" layer="16"/>
+<wire x1="15.25" y1="63.75" x2="15.25" y2="70" width="0.1524" layer="16"/>
+<wire x1="17" y1="50.581" x2="16.5" y2="51.081" width="0.1524" layer="16"/>
+<wire x1="16.5" y1="51.081" x2="16.5" y2="62.5" width="0.1524" layer="16"/>
 </signal>
 <signal name="ENC1PINB">
 <contactref element="ENC1" pad="B"/>
 <contactref element="U$1" pad="21/A7"/>
-<wire x1="19.376" y1="48.041" x2="15.74" y2="48.041" width="0.1524" layer="16"/>
-<wire x1="15.74" y1="48.041" x2="15.74" y2="61.76" width="0.1524" layer="16"/>
-<wire x1="14" y1="63.5" x2="14" y2="68" width="0.1524" layer="16"/>
-<wire x1="14" y1="68" x2="11.427" y2="68" width="0.1524" layer="16"/>
+<wire x1="19.376" y1="48.041" x2="16.5" y2="48.041" width="0.1524" layer="16"/>
+<wire x1="14.25" y1="62.75" x2="14.25" y2="68" width="0.1524" layer="16"/>
+<wire x1="14.25" y1="68" x2="11.427" y2="68" width="0.1524" layer="16"/>
 <wire x1="11.427" y1="68" x2="11.235" y2="68.192" width="0.1524" layer="16"/>
-<wire x1="15.74" y1="61.76" x2="14" y2="63.5" width="0.1524" layer="16"/>
+<wire x1="15.74" y1="61.26" x2="14.25" y2="62.75" width="0.1524" layer="16"/>
+<wire x1="16.5" y1="48.041" x2="15.74" y2="48.801" width="0.1524" layer="16"/>
+<wire x1="15.74" y1="48.801" x2="15.74" y2="61.26" width="0.1524" layer="16"/>
 </signal>
 <signal name="ENC2SW">
@@
 <wire x1="5.4938" y1="61.4364" x2="11.9962" y2="61.4364" width="0.1524" layer="16"/>
 <contactref element="U$1" pad="20/A6"/>
-<wire x1="11.9962" y1="61.4364" x2="15" y2="58.4326" width="0.1524" layer="16"/>
-<wire x1="15" y1="58.4326" x2="15" y2="45.5" width="0.1524" layer="16"/>
-<wire x1="15" y1="45.5" x2="19.375" y2="45.5" width="0.1524" layer="16"/>
+<wire x1="15" y1="58.4326" x2="11.9962" y2="61.4364" width="0.1524" layer="16"/>
+<wire x1="19.375" y1="45.5" x2="15.5" y2="45.5" width="0.1524" layer="16"/>
 <wire x1="19.375" y1="45.5" x2="19.376" y2="45.501" width="0.1524" layer="16"/>
+<wire x1="15.5" y1="45.5" x2="15" y2="46" width="0.1524" layer="16"/>
+<wire x1="15" y1="46" x2="15" y2="58.4326" width="0.1524" layer="16"/>
 </signal>
 <signal name="B2">
@@
 <contactref element="R10" pad="1"/>
 <wire x1="8.5" y1="58" x2="8.5" y2="57.95" width="0.1524" layer="16"/>
-<wire x1="3.95" y1="55" x2="3.85" y2="57.35" width="0.1524" layer="16"/>
-<wire x1="3.85" y1="57.35" x2="4.5" y2="58" width="0.1524" layer="16"/>
 <wire x1="4.5" y1="58" x2="8.5" y2="58" width="0.1524" layer="16"/>
 <contactref element="U$1" pad="17/A3"/>
@@
 <wire x1="16.65" y1="44.35" x2="15.75" y2="45.25" width="0.1524" layer="1"/>
 <wire x1="10" y1="45.25" x2="10" y2="57.5" width="0.1524" layer="1"/>
+<wire x1="3.95" y1="55" x2="3.95" y2="57.45" width="0.1524" layer="16"/>
+<wire x1="3.95" y1="57.45" x2="4.5" y2="58" width="0.1524" layer="16"/>
 </signal>
 <signal name="CVIN2">
@@
 <wire x1="12.5" y1="47.865" x2="13.905" y2="46.46" width="0.1524" layer="1"/>
 <wire x1="12.5" y1="47.865" x2="12.5" y2="58.5" width="0.1524" layer="1"/>
-<wire x1="12.5" y1="58.5" x2="14" y2="60" width="0.1524" layer="1"/>
-<wire x1="14" y1="60" x2="14" y2="71" width="0.1524" layer="1"/>
+<wire x1="12.5" y1="58.5" x2="14.5" y2="60.5" width="0.1524" layer="1"/>
+<wire x1="14.5" y1="60.5" x2="14.5" y2="70.5" width="0.1524" layer="1"/>
 <wire x1="11.5" y1="73.5" x2="11.5" y2="79.5" width="0.1524" layer="1"/>
 <wire x1="11.5" y1="79.5" x2="12.5" y2="80.5" width="0.1524" layer="1"/>
-<wire x1="14" y1="71" x2="11.5" y2="73.5" width="0.1524" layer="1"/>
+<wire x1="14.5" y1="70.5" x2="11.5" y2="73.5" width="0.1524" layer="1"/>
 <wire x1="12.5" y1="86" x2="11" y2="87.5" width="0.1524" layer="1"/>
 </signal>

Commit message: pcb and pannel revision
Parts:
- moved D1 1.50 mm to (6.95, 24.4)
- moved CV1 0.50 mm to (25.0, 90.5)
- moved CV2 0.50 mm to (35.1, 90.5)
- moved CV3 0.50 mm to (45.1, 90.5)
- moved CV4 0.50 mm to (55.1, 90.5)
- moved IN1 0.50 mm to (4.95, 103.5)
- moved IN2 0.50 mm to (15.0, 103.5)
- moved IN3 0.50 mm to (4.95, 90.5)
- moved IN4 0.50 mm to (15.0, 90.5)
- moved R1 0.50 mm to (10.0, 104.0)
- moved R13 0.50 mm to (30.0, 104.0)
- moved R14 0.50 mm to (40.0, 104.0)
- moved R15 0.50 mm to (56.8, 104.0)
- moved R18 0.50 mm to (36.8, 90.0)
- moved R2 0.50 mm to (20.0, 104.0)
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Routing:
- net VCC: track 76.0 -> 78.8 mm
- net N$1: track 5.29 -> 6.79 mm
- net GND: track 601.5 -> 603.0 mm
- net N$24: track 63.2 -> 62.1 mm
- net ENC2PINB: track 37.9 -> 38.5 mm
- net OLEDRST: track 51.0 -> 51.5 mm
- net OLEDDATA: track 64.6 -> 65.1 mm
- net OLEDCS: track 60.4 -> 60.9 mm
- net OLEDCLK: track 60.8 -> 61.3 mm
- net N$7: track 73.9 -> 74.4 mm
- net N$39: track 64.2 -> 64.7 mm
- net N$37: track 84.8 -> 85.3 mm
- net N$31: track 65.6 -> 66.1 mm
- net N$27: track 44.1 -> 44.6 mm
- net N$21: track 60.8 -> 61.3 mm
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Other:
- board size 60 x 110 mm -> 60 x 110.5 mm

Commit message: superposition
Parts:
- R5, R6, R7, R8: value 100k -> 56k
Changed lines of the file:
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@@
 <drawing>
 <settings>
-<setting alwaysvectorfont="yes"/>
+<setting alwaysvectorfont="no"/>
 <setting verticaltext="up"/>
 </settings>
@@
 <attribute name="VALUE" x="43.714" y="55.238" size="1.27" layer="28" rot="MR90"/>
 </element>
-<element name="R5" library="rcl" library_urn="urn:adsk.eagle:library:334" package="R0805" package3d_urn="urn:adsk.eagle:package:23553/2" value="100k" x="8.5" y="57" smashed="yes" rot="MR270">
+<element name="R5" library="rcl" library_urn="urn:adsk.eagle:library:334" package="R0805" package3d_urn="urn:adsk.eagle:package:23553/2" value="56k" x="8.5" y="57" smashed="yes" rot="MR270">
 <attribute name="NAME" x="7.484" y="57.762" size="1.27" layer="26" rot="MR270"/>
 <attribute name="SPICEPREFIX" value="R" x="8.5" y="57" size="1.778" layer="28" rot="MR270" display="off"/>
 <attribute name="VALUE" x="11.286" y="58.262" size="1.27" layer="28" rot="MR270"/>
 </element>
-<element name="R6" library="rcl" library_urn="urn:adsk.eagle:library:334" package="R0805" package3d_urn="urn:adsk.eagle:package:23553/2" value="100k" x="10" y="51.5" smashed="yes" rot="MR90">
+<element name="R6" library="rcl" library_urn="urn:adsk.eagle:library:334" package="R0805" package3d_urn="urn:adsk.eagle:package:23553/2" value="56k" x="10" y="51.5" smashed="yes" rot="MR90">
 <attribute name="NAME" x="11.016" y="50.738" size="1.27" layer="26" rot="MR90"/>
 <attribute name="SPICEPREFIX" value="R" x="10" y="51.5" size="1.778" layer="28" rot="MR90" display="off"/>
 <attribute name="VALUE" x="7.714" y="50.738" size="1.27" layer="28" rot="MR90"/>
 </element>
-<element name="R7" library="rcl" library_urn="urn:adsk.eagle:library:334" package="R0805" package3d_urn="urn:adsk.eagle:package:23553/2" value="100k" x="8.5" y="46" smashed="yes" rot="MR270">
+<element name="R7" library="rcl" library_urn="urn:adsk.eagle:library:334" package="R0805" package3d_urn="urn:adsk.eagle:package:23553/2" value="56k" x="8.5" y="46" smashed="yes" rot="MR270">
 <attribute name="NAME" x="7.484" y="47.262" size="1.27" layer="26" rot="MR270"/>
 <attribute name="SPICEPREFIX" value="R" x="8.5" y="46" size="1.778" layer="28" rot="MR270" display="off"/>
 <attribute name="VALUE" x="10.786" y="46.762" size="1.27" layer="28" rot="MR270"/>
 </element>
-<element name="R8" library="rcl" library_urn="urn:adsk.eagle:library:334" package="R0805" package3d_urn="urn:adsk.eagle:package:23553/2" value="100k" x="8.5" y="40.5" smashed="yes" rot="MR270">
+<element name="R8" library="rcl" library_urn="urn:adsk.eagle:library:334" package="R0805" package3d_urn="urn:adsk.eagle:package:23553/2" value="56k" x="8.5" y="40.5" smashed="yes" rot="MR270">
 <attribute name="NAME" x="7.484" y="40.762" size="1.27" layer="26" rot="MR270"/>
 <attribute name="SPICEPREFIX" value="R" x="8.5" y="40.5" size="1.778" layer="28" rot="MR270" display="off"/>
