File: HardWare/Pannel/SP_Pannel.brd (EAGLE design)
At the start: 60.6 x 128.5 mm, 0 parts

Commit message: added gerber files
Changed lines of the file:
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@@
 <dimension x1="-7.47" y1="119.28" x2="-7.47" y2="128.53" x3="-7.47" y3="123.905" textsize="1.778" layer="1"/>
 <dimension x1="0.03" y1="-3.47" x2="53.25" y2="-3.46" x3="26.639996875" y3="-3.465" textsize="1.778" layer="1"/>
-<text x="23.33" y="124.03" size="1.778" layer="25">SuperPosition</text>
+<text x="23.33" y="124.53" size="1.778" layer="25">SuperPosition</text>
 <dimension x1="0.03" y1="-6.72" x2="7.53" y2="-6.72" x3="3.78" y3="-6.72" textsize="1.778" layer="1"/>
 <hole x="5.25" y="112.25" drill="6" locked="yes"/>
@@
 <text x="33" y="9" size="1.778" layer="25">15</text>
 <text x="48" y="9" size="1.778" layer="25">16</text>
+<hole x="30.3" y="54.25" drill="2.8"/>
+<hole x="30.3" y="24.25" drill="2.8"/>
 </plain>
 <attributes>
