File: HardWare/Pannel/SP_Pannel.brd (EAGLE design)
At the start: 60.6 x 128.5 mm, 0 parts

Commit message: pcb and pannel revision
Other:
- outline, holes or cut-outs redrawn
- board text added: "SuperPosition"
